File: ADAU1701/freeDSP.sch (EAGLE design)
At the start: 122 parts, among them IC1 24AA256P, IC2 REG1117, IC3 AD8608R, Q1 12.288Mhz, Q2 2N7000, Q3 2N7000, Q4 2N7000, Q5 2N7000, T1 FZT751TA, X1 TOBU3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

Commit message: Add Atmega32 DIP40
Other:
- moved on the sheet: C1, C10, C11, C12, C13, C14, C15, C16, C17, C18, C19, C2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

Commit message: add pcb image
Other:
- note removed: "This work and all other materials under https://github.com/freeDSP are licensed under a Creative Commons Attribution Share-Alike 4.0 license. This allows for both personal and commercial derivative works, as long as they credit freeDSP and release their designs under the same license."
Changed lines of the file:
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@@
 <text x="358.14" y="40.64" size="5.08" layer="91">freeDSP 1.1
 www.freedsp.cc</text>
-<text x="40.64" y="215.9" size="2.54" layer="91" font="vector" distance="100">This work and all other materials
-under https://github.com/freeDSP
-are licensed under a Creative Commons
-Attribution Share-Alike 4.0 license.
-This allows for both personal and
-commercial derivative works, as long
-as they credit freeDSP and release
-their designs under the same license.</text>
 </plain>
 <instances>
@@
 </sheet>
 </sheets>
-<errors>
-</errors>
 </schematic>
 </drawing>
