File: Atmega32/Dip40-Extend/Development Board ATMega32.sch (EAGLE design)
At the start: 63 parts, among them IC1 REG1117, IC2 MEGA32-P, IC3 7805T, P1 PIN-BIG1X, P10 PIN-BIG1X, P11 PIN-BIG1X, P12 PIN-BIG1X, P13 PIN-BIG1X, P14 PIN-BIG1X, P15 PIN-BIG1X, P16 PIN-BIG1X, P17 PIN-BIG1X, P18 PIN-BIG1X, P19 PIN-BIG1X, P2 PIN-BIG1X, P20 PIN-BIG1X, P21 PIN-BIG1X, P22 PIN-BIG1X, P23 PIN-BIG1X, P24 PIN-BIG1X, P25 PIN-BIG1X, P26 PIN-BIG1X, P3 PIN-BIG1X, P4 PIN-BIG1X, P5 PIN-BIG1X, P6 PIN-BIG1X, P7 PIN-BIG1X, P8 PIN-BIG1X, P9 PIN-BIG1X, Q3 16m, SW2 smd_sw, X1 PN61729-S, X3 057-010-1

Commit message: update Atemga32 Extends Dip40
Parts:
- renumbered FTDI to SERIAL
Other:
- note added: "ADDITIONAL NEXTION HEADER"
- note added: "I2C PINS"
- note added: "NEXTION HEADER"
- note added: "VIN REGULATOR"
- note added: "X3-3 is not used"
- note removed: "DISPLAY HEADER"
- moved on the sheet: C1, C10, C11, C2, C3, C4, C5, D1, IC1, IC3, LED_13, P1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
